Commit message: 1227

File: wheeltec_robot_urdf/wheeltec_robot_urdf/urdf/mini_mec_robot.urdf (robot description, URDF)
Before this commit: robot wheeltec_robot, 6 links, 5 joints
Links:
- link base_link: geometry visual box size=1.08 0.76 0.05
- link left_front_link: geometry visual cylinder length=0.073 radius=0.09
- link left_wheel_link: geometry visual cylinder length=0.073 radius=0.09
- link right_front_link: geometry visual cylinder length=0.073 radius=0.09
- link right_wheel_link: geometry visual cylinder length=0.073 radius=0.09
Joints:
- joint left_front_joint: axis 0 1 0 -> 0 0 1; origin xyz=0.085 0.0975 0.0375 rpy=1.57 0 0 -> xyz=0.325 0.3285 0.09 rpy=-1.57 0 0
- joint left_wheel_joint: axis 0 1 0 -> 0 0 1; origin xyz=-0.085 0.0975 0.0375 rpy=1.57 0 0 -> xyz=-0.325 0.3285 0.09 rpy=-1.57 0 0
- joint right_front_joint: axis 0 1 0 -> 0 0 1; origin xyz=0.085 -0.0975 0.0375 rpy=1.57 0 0 -> xyz=0.325 -0.3285 0.09 rpy=-1.57 0 0
- joint right_wheel_joint: axis 0 1 0 -> 0 0 1; origin xyz=-0.085 -0.0975 0.0375 rpy=1.57 0 0 -> xyz=-0.325 -0.3285 0.09 rpy=-1.57 0 0

Commit message: 0114backup

File: wheeltec_robot_urdf/wheeltec_robot_urdf/urdf/mini_mec_robot.urdf (robot description, URDF)
Before this commit: robot wheeltec_robot, 6 links, 5 joints
Joints:
- joint left_front_joint: origin xyz=0.325 0.3285 0.09 rpy=-1.57 0 0 -> xyz=0.325 0.3285 0.09 rpy=1.57 0 0
- joint left_wheel_joint: origin xyz=-0.325 0.3285 0.09 rpy=-1.57 0 0 -> xyz=-0.325 0.3285 0.09 rpy=1.57 0 0
- joint right_front_joint: origin xyz=0.325 -0.3285 0.09 rpy=-1.57 0 0 -> xyz=0.325 -0.3285 0.09 rpy=1.57 0 0
- joint right_wheel_joint: origin xyz=-0.325 -0.3285 0.09 rpy=-1.57 0 0 -> xyz=-0.325 -0.3285 0.09 rpy=1.57 0 0
